File: OLED_096_SH1101A_main.brd (EAGLE design)
At the start: 27.9 x 31.7 mm, 47 parts, among them IC1 MEGA8-AI, IC2 78L05Z, Q1 SI2302, Q2 BC847ASMD, Q3 BC847ASMD, Q4 BC857ASMD

Commit message: Fix schematic
Parts:
- removed JP1, JP2: (no value), SparkFun:1X08
- added D3, D4: (no value), diode:MINIMELF
- D2: value (none) -> 2.5V
- moved S1 169.3 mm to (49.8, 26.6), turned to 90 degrees
- moved LED1 166.9 mm to (51.0, 20.5)
- moved C11 162.6 mm to (52.4, 2.33), turned to 90 degrees
- moved R20 160.9 mm to (35.5, 1.87), turned to 180 degrees
- moved IC2 155.8 mm to (47.3, 2.02)
- moved C10 148.8 mm to (38.4, 11.5)
- moved C9 142.4 mm to (49.3, 6.07)
- moved R19 137.2 mm to (38.1, 18.0)
- moved R18 135.5 mm to (38.7, 21.6), turned to 180 degrees
- moved Q4 134.8 mm to (42.8, 7.31)
- moved R17 134.3 mm to (43.1, 24.3)
- moved R16 119.1 mm to (42.8, 13.4)
- moved R15 104.1 mm to (42.8, 2.02), turned to 180 degrees
- moved Q3 102.4 mm to (49.3, 10.1)
- moved Q2 101.2 mm to (47.6, 17.1)
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Connections:
- net +3V3: now also D3.A; no longer JP1.2
- net GND: now also C10.2, C11.2, C9.2, IC2.2, Q3.2, R17.1; no longer JP1.1
- net N$15: now also D3.C, D4.A; no longer C10.2, C11.2, C9.2, IC2.2, Q3.2, R17.1
- net OLED_A0: no longer JP1.6
- net OLED_CS: no longer JP1.4
- net OLED_D0(SCK): no longer JP2.1
- net OLED_D1(SDI): no longer JP2.2
- net OLED_D2: no longer JP2.3
- net OLED_D3: no longer JP2.4
- net OLED_D4: no longer JP2.5
- net OLED_D5: no longer JP2.6
- net OLED_D6: no longer JP2.7
- net OLED_D7: no longer JP2.8
- net OLED_RD: no longer JP1.8
- net OLED_RES: no longer JP1.5
- net OLED_WR: no longer JP1.7
- net P/S: no longer JP1.3
- net VCC: now also D4.C
Routing:
- net OLED_RES: track 33.9 -> 0.00 mm, vias 2 -> 0
- net OLED_RD: track 28.3 -> 0.00 mm, vias 3 -> 0
- net OLED_A0: track 27.6 -> 0.00 mm, vias 1 -> 0
- net OLED_WR: track 21.4 -> 0.00 mm, vias 2 -> 0
- net OLED_D0(SCK): track 19.1 -> 0.02 mm
- net OLED_D1(SDI): track 16.8 -> 0.02 mm
- net OLED_CS: track 18.6 -> 2.18 mm
- net P/S: track 19.9 -> 3.81 mm
- net OLED_D2: track 15.0 -> 0.00 mm
- net OLED_D3: track 13.2 -> 0.00 mm
- net OLED_D4: track 11.0 -> 0.00 mm
- net OLED_D7: track 10.5 -> 0.00 mm
- net OLED_D5: track 10.2 -> 0.00 mm
- net GND: track 14.2 -> 4.14 mm, vias 3 -> 0
- net OLED_D6: track 9.68 -> 0.00 mm
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Other:
- board size 27.9 x 31.7 mm -> 53.3 x 33.9 mm
- board text removed: "+3.3V"
- board text removed: "/CS"
- board text removed: "/RST"
- board text removed: "A0"
- board text removed: "D0(SCK)"
- board text removed: "D1(SDI)"
- board text removed: "D2"
- board text removed: "D3"
- board text removed: "D4"
- board text removed: "D5"
- board text removed: "D6"
- board text removed: "D7"
- board text removed: "GND"
- board text removed: "P/S"
- board text removed: "RD"
- board text removed: "WR"
