File: OLED_096_SH1101A_main.sch (EAGLE design)
At the start: 47 parts, among them IC1 MEGA8-AI, IC2 78L05Z, Q1 SI2302, Q2 BC847ASMD, Q3 BC847ASMD, Q4 BC857ASMD

Commit message: Fix schematic
Parts:
- removed JP1, JP2: (no value), SparkFun:M08
- added D3, D4: (no value), diode:DIODE-MINIMELF
- D2: value (none) -> 2.5V
Connections:
- net +3V3: now also D3.A; no longer JP1.2
- net GND: now also C10.2, C11.2, C9.2, IC2.GND, Q3.E, R17.1; no longer JP1.1
- net N$15: now also D3.C, D4.A; no longer C10.2, C11.2, C9.2, IC2.GND, Q3.E, R17.1
- net OLED_A0: no longer JP1.6
- net OLED_CS: no longer JP1.4
- net OLED_D0(SCK): no longer JP2.1
- net OLED_D1(SDI): no longer JP2.2
- net OLED_D2: no longer JP2.3
- net OLED_D3: no longer JP2.4
- net OLED_D4: no longer JP2.5
- net OLED_D5: no longer JP2.6
- net OLED_D6: no longer JP2.7
- net OLED_D7: no longer JP2.8
- net OLED_RD: no longer JP1.8
- net OLED_RES: no longer JP1.5
- net OLED_WR: no longer JP1.7
- net P/S: no longer JP1.3
- net VCC: now also D4.C
Other:
- moved on the sheet: C7, C8, D2, JP3, Q2, R10, R11, R12, R13, R14, R19, R20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
